File: power.kicad_sch (KiCad schematic)
At the start: 19 parts, among them J6 VBUS_EXT, Q2 GSFF3134, U2 LMS3635LQURNLRQ1

Commit message: fix erc errors
Changed lines of the file:
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@@
 	)
 	(junction
-		(at 166.37 93.98)
-		(diameter 0)
-		(color 0 0 0 0)
-	)
-	(junction
 		(at 97.79 77.47)
 		(diameter 0)
@@
 	(wire
 		(pts
-			(xy 166.37 93.98) (xy 166.37 107.95)
+			(xy 166.37 85.09) (xy 166.37 107.95)
 		)
 		(stroke
@@
 	(wire
 		(pts
-			(xy 166.37 85.09) (xy 166.37 93.98)
-		)
-		(stroke
-			(width 0)
-			(type default)
-		)
-	)
-	(wire
-		(pts
 			(xy 109.22 77.47) (xy 97.79 77.47)
 		)
@@
 					(unit 1)
 				)
-			)
-		)
-	)
-	(symbol
-		(lib_id "power:PWR_FLAG")
-		(at 166.37 93.98 270)
-		(unit 1)
-		(exclude_from_sim no)
-		(in_bom yes)
-		(on_board yes)
-		(dnp no)
-		(property "Reference" "#FLG01"
-			(at 168.275 93.98 0)
-			(effects
-				(font
-					(size 1.27 1.27)
-				)
-				(hide yes)
-			)
-		)
-		(property "Value" "PWR_FLAG"
-			(at 170.18 93.9801 90)
-			(effects
-				(font
-					(size 1.27 1.27)
-				)
-				(justify left)
-			)
-		)
-		(property "Footprint" ""
-			(at 166.37 93.98 0)
-			(effects
-				(font
-					(size 1.27 1.27)
-				)
-				(hide yes)
-			)
-		)
-		(property "Datasheet" "~"
-			(at 166.37 93.98 0)
-			(effects
-				(font
-					(size 1.27 1.27)
-				)
-				(hide yes)
-			)
-		)
-		(property "Description" "Special symbol for telling ERC where power comes from"
-			(at 166.37 93.98 0)
-			(effects
-				(font
-					(size 1.27 1.27)
-				)
-				(hide yes)
-			)
-		)
-		(pin "1"
-		)
-		(instances
-			(project "effectiveRangeRelay"
-				(path "/6eab7a25-9b20-4eb7-9336-dd2042abdd78/23c81081-336d-40d7-9598-c756c6e0c615"
-					(reference "#FLG01")
-					(unit 1)
-				)
