File: power.kicad_sch (KiCad schematic)
At the start: 19 parts, among them J6 VBUS_EXT, Q2 GSFF3134, U2 LMS3635LQURNLRQ1

Commit message: fix drc errors
Parts:
- C8: MPN GRM155R71E104KE14J -> GRM155R61H474ME11D; SupplierLink https://www.digikey.hu/en/products/detail/murata-electronic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 -> https://www.digikey.com/en/products/detail/murata-electroni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
Changed lines of the file:
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@@
 			)
 		)
-		(property "MPN" "GRM155R71E104KE14J"
+		(property "MPN" "GRM155R61H474ME11D"
 			(at 173.99 72.39 0)
 			(effects
@@
 			)
 		)
-		(property "SupplierLink" "https://www.digikey.hu/en/products/detail/murata-electronics/GRM188R72A104KA35D/702549"
+		(property "SupplierLink" "https://www.digikey.com/en/products/detail/murata-electronics/GRM155R61H474ME11D/10694674"
 			(at 173.99 72.39 0)
 			(effects
